Commit message: base_scan2(2번 라이다)위치 수정 적용

File: urdf/stella.urdf (robot description, URDF)
Before this commit: robot stella, 5 links, 4 joints
Joints:
- joint scan2_joint: origin xyz=0.202 0.0 0.032 rpy=0.0 0.0 -1.57 -> xyz=-0.166 0.0 0.223 rpy=0.0 0.0 3.1415

File: urdf/stella_realsense.urdf (robot description, URDF)
Before this commit: robot stella, 6 links, 5 joints
Joints:
- joint scan2_joint: origin xyz=0.202 0.0 0.032 rpy=0.0 0.0 -1.57 -> xyz=-0.166 0.0 0.223 rpy=0.0 0.0 3.1415

File: urdf/stella_web_cam.urdf (robot description, URDF)
Before this commit: robot stella, 6 links, 5 joints
Joints:
- joint scan2_joint: origin xyz=0.202 0.0 0.032 rpy=0.0 0.0 -1.57 -> xyz=-0.166 0.0 0.223 rpy=0.0 0.0 3.1415
